Commit message: bug fixed

File: load_runner_description/urdf/load_runner_300lt.urdf.xacro (robot description, xacro)
@@ -194,5 +194,5 @@
                     <geometry>
                         <!-- <mesh filename="package://load_runner_description/meshes/load_runner_300lt/caster_wheel.stl" scale="1 1 1"/> -->
-                        <cylinder radius="0.03746" length="0.023"/>
+                        <cylinder radius="0.0373" length="0.023"/>
                     </geometry>
                 </collision>
@@ -220,5 +220,5 @@
                     <geometry>
                         <!-- <mesh filename="package://load_runner_description/meshes/load_runner_300lt/caster_wheel.stl" scale="1 1 1"/> -->
-                        <cylinder radius="0.03746" length="0.023"/>
+                        <cylinder radius="0.0373" length="0.023"/>
                     </geometry>
                 </collision>
